File: SLACRnStill-V2/nEXO_pcbV2/Official level sensorV2.kicad_pcb (KiCad board)
At the start: 2 copper layers, 101.6 x 78.2 mm, 34 parts, among them J1 Conn_01x02_Male, J10 70543-0003, J2 Conn_01x04_Female, J3 M05PTH, J4 440055-4, J5 M05PTH, J6 70543-0003, J7 70543-0003, J8 70543-0003, J9 70543-0003, P10 CONN_01X01, P11 CONN_01X01, P12 CONN_01X01, P13 CONN_01X01, P2 Power, P4 Analog, P5 PWM, P6 PWM, P8 CONN_01X01, P9 CONN_01X01, U1 AD7151

Commit message: I adressed issue #1
Parts:
- J10, J6, J7, J8, J9: footprint Connector:SHDR4W97P0X254_1X4_1271X660X1143P -> SparkFun_LoadCell:SHDR4W97P0X254_1X4_1271X660X1143P
- J4: footprint Connector:TE_440055-4 -> SparkFun_LoadCell:SHDR4W97P0X254_1X4_1271X660X1143P
- moved J9 4.53 mm to (134.1, 49.5)
- moved J10 4.53 mm to (134.1, 61.2)
- moved J7 3.85 mm to (111.2, 61.4)
- moved J6 3.84 mm to (111.2, 49.7)
- moved J4 3.09 mm to (109.4, 78.0)
- moved J8 2.70 mm to (122.8, 55.7)
Routing:
- net Net-(J3-Pad5): track 20.9 -> 14.2 mm
- net Net-(J3-Pad4): track 20.3 -> 14.2 mm
- net Net-(J3-Pad3): track 20.1 -> 14.2 mm
- net Net-(J3-Pad2): track 19.6 -> 14.2 mm
- net Net-(J10-Pad3): track 72.8 -> 76.4 mm
- net Net-(J10-Pad4): track 71.1 -> 74.4 mm
- net Net-(J10-Pad1): track 46.7 -> 48.1 mm
- net Net-(J10-Pad2): track 62.8 -> 63.8 mm
