File: SLACRnStill-V2/nEXO_pcbV2/Official level sensorV2.kicad_sch (KiCad schematic)
At the start: 32 parts, among them J1 Conn_01x02_Male, J10 70543-0003, J2 Conn_01x04_Female, J3 M05PTH, J4 440055-4, J5 M05PTH, J6 70543-0003, J7 70543-0003, J8 70543-0003, J9 70543-0003, P10 CONN_01X01, P11 CONN_01X01, P12 CONN_01X01, P13 CONN_01X01, P2 Power, P4 Analog, P5 PWM, P6 PWM, P8 CONN_01X01, P9 CONN_01X01, U1 AD7151

Commit message: I adressed issue #1
Parts:
- J10, J6, J7, J8, J9: footprint Connector:SHDR4W97P0X254_1X4_1271X660X1143P -> SparkFun_LoadCell:SHDR4W97P0X254_1X4_1271X660X1143P
- J4: footprint Connector:TE_440055-4 -> SparkFun_LoadCell:SHDR4W97P0X254_1X4_1271X660X1143P
Changed lines of the file:
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@@
       (effects (font (size 1.27 1.27)) (justify left))
     )
-    (property "Footprint" "Connector:SHDR4W97P0X254_1X4_1271X660X1143P" (id 2) (at 369.57 165.1 0)
+    (property "Footprint" "SparkFun_LoadCell:SHDR4W97P0X254_1X4_1271X660X1143P" (id 2) (at 369.57 165.1 0)
       (effects (font (size 1.27 1.27)) (justify left) hide)
     )
@@
       (effects (font (size 1.27 1.27)) (justify left))
     )
-    (property "Footprint" "Connector:TE_440055-4" (id 2) (at 480.06 346.71 0)
+    (property "Footprint" "SparkFun_LoadCell:SHDR4W97P0X254_1X4_1271X660X1143P" (id 2) (at 480.06 346.71 0)
       (effects (font (size 1.27 1.27)) (justify left bottom) hide)
     )
@@
       (effects (font (size 1.27 1.27)) (justify left))
     )
-    (property "Footprint" "Connector:SHDR4W97P0X254_1X4_1271X660X1143P" (id 2) (at 342.9 177.8 0)
+    (property "Footprint" "SparkFun_LoadCell:SHDR4W97P0X254_1X4_1271X660X1143P" (id 2) (at 342.9 177.8 0)
       (effects (font (size 1.27 1.27)) (justify left) hide)
     )
@@
       (effects (font (size 1.27 1.27)) (justify left))
     )
-    (property "Footprint" "Connector:SHDR4W97P0X254_1X4_1271X660X1143P" (id 2) (at 342.9 152.4 0)
+    (property "Footprint" "SparkFun_LoadCell:SHDR4W97P0X254_1X4_1271X660X1143P" (id 2) (at 342.9 152.4 0)
       (effects (font (size 1.27 1.27)) (justify left) hide)
     )
@@
       (effects (font (size 1.27 1.27)) (justify left))
     )
-    (property "Footprint" "Connector:SHDR4W97P0X254_1X4_1271X660X1143P" (id 2) (at 394.97 177.8 0)
+    (property "Footprint" "SparkFun_LoadCell:SHDR4W97P0X254_1X4_1271X660X1143P" (id 2) (at 394.97 177.8 0)
       (effects (font (size 1.27 1.27)) (justify left) hide)
     )
@@
       (effects (font (size 1.27 1.27)) (justify left))
     )
-    (property "Footprint" "Connector:SHDR4W97P0X254_1X4_1271X660X1143P" (id 2) (at 394.97 152.4 0)
+    (property "Footprint" "SparkFun_LoadCell:SHDR4W97P0X254_1X4_1271X660X1143P" (id 2) (at 394.97 152.4 0)
       (effects (font (size 1.27 1.27)) (justify left) hide)
     )
@@
     )
     (path "/32c7f27c-409f-4394-a15b-7d9d637c8644"
-      (reference "J4") (unit 1) (value "440055-4") (footprint "Connector:TE_440055-4")
+      (reference "J4") (unit 1) (value "440055-4") (footprint "SparkFun_LoadCell:SHDR4W97P0X254_1X4_1271X660X1143P")
     )
     (path "/f5b068dd-8254-49a7-83b7-cfb8c277fd17"
@@
     )
     (path "/9811e649-d0e3-4b4a-a0f2-65f71120d5b6"
-      (reference "J6") (unit 1) (value "70543-0003") (footprint "Connector:SHDR4W97P0X254_1X4_1271X660X1143P")
+      (reference "J6") (unit 1) (value "70543-0003") (footprint "SparkFun_LoadCell:SHDR4W97P0X254_1X4_1271X660X1143P")
     )
     (path "/372dddc1-cb4f-4294-9fc4-ca7f615d3d36"
-      (reference "J7") (unit 1) (value "70543-0003") (footprint "Connector:SHDR4W97P0X254_1X4_1271X660X1143P")
+      (reference "J7") (unit 1) (value "70543-0003") (footprint "SparkFun_LoadCell:SHDR4W97P0X254_1X4_1271X660X1143P")
     )
     (path "/1224341a-7e93-4268-a280-9be512693515"
-      (reference "J8") (unit 1) (value "70543-0003") (footprint "Connector:SHDR4W97P0X254_1X4_1271X660X1143P")
+      (reference "J8") (unit 1) (value "70543-0003") (footprint "SparkFun_LoadCell:SHDR4W97P0X254_1X4_1271X660X1143P")
     )
     (path "/c12e1fb7-ff4d-4c24-958d-1d48ec6dcceb"
-      (reference "J9") (unit 1) (value "70543-0003") (footprint "Connector:SHDR4W97P0X254_1X4_1271X660X1143P")
+      (reference "J9") (unit 1) (value "70543-0003") (footprint "SparkFun_LoadCell:SHDR4W97P0X254_1X4_1271X660X1143P")
     )
     (path "/b31c638f-24bf-4d28-a633-fb04793fcc0c"
-      (reference "J10") (unit 1) (value "70543-0003") (footprint "Connector:SHDR4W97P0X254_1X4_1271X660X1143P")
+      (reference "J10") (unit 1) (value "70543-0003") (footprint "SparkFun_LoadCell:SHDR4W97P0X254_1X4_1271X660X1143P")
     )
     (path "/5ae7cb3b-55c5-4184-85ac-b02dab9de08f"
